File: eagle/Actuator Circle.sch (EAGLE design)
At the start: 28 parts, among them Q1 FDV301N

Commit message: Modified Resistors to 0603, and moved them to the same side
Modified Resistors to 0603, and moved them to the same side, so as to make assembly slightly easier.
Parts:
- R2, R3, R4, R5, R6: device Actuator Circle:RES-0402 -> resistor:R-EU_R0603
Changed lines of the file:
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@@
 <?xml version="1.0" encoding="utf-8"?>
 <!DOCTYPE eagle SYSTEM "eagle.dtd">
-<eagle version="9.4.2">
+<eagle version="9.3.0">
 <drawing>
 <settings>
@@
 <part name="Q1" library="Actuator Circle" deviceset="SMD-MOSFET-N-CH-25V-220MA-FDV301N(SOT-23)" device="" package3d_urn="urn:adsk.eagle:package:28738/2" value="FDV301N"/>
 <part name="D1" library="Actuator Circle" deviceset="D-" device="SOD123" package3d_urn="urn:adsk.eagle:package:26308/2" value="1N4148W-7-F"/>
-<part name="R3" library="Actuator Circle" deviceset="RES-0402" device="" package3d_urn="urn:adsk.eagle:package:10872901/3" value="100Ohm"/>
-<part name="R4" library="Actuator Circle" deviceset="RES-0402" device="" package3d_urn="urn:adsk.eagle:package:10872901/3" value="1MOhm"/>
+<part name="R3" library="resistor" library_urn="urn:adsk.eagle:library:348" deviceset="R-EU_" device="R0603" package3d_urn="urn:adsk.eagle:package:23555/3" value="100Ohm"/>
+<part name="R4" library="resistor" library_urn="urn:adsk.eagle:library:348" deviceset="R-EU_" device="R0603" package3d_urn="urn:adsk.eagle:package:23555/3" value="1MOhm"/>
 <part name="C1" library="BeagleBone_Blue_R3" library_urn="urn:adsk.eagle:library:5828899" deviceset="CAPACITOR-P" device="E2.5-6" package3d_urn="urn:adsk.eagle:package:5829619/1" value="100UF"/>
 <part name="LED1" library="Actuator Circle" deviceset="LED" device="CHIPLED_0805" package3d_urn="urn:adsk.eagle:package:15821/2" value="17-21SURC/S530-A3/TR8"/>
-<part name="R2" library="Actuator Circle" deviceset="RES-0402" device="" package3d_urn="urn:adsk.eagle:package:10872901/3" value="1K"/>
+<part name="R2" library="resistor" library_urn="urn:adsk.eagle:library:348" deviceset="R-EU_" device="R0603" package3d_urn="urn:adsk.eagle:package:23555/3" value="1K"/>
 <part name="LED2" library="Actuator Circle" deviceset="LED" device="CHIPLED_0805" package3d_urn="urn:adsk.eagle:package:15821/2" value="17-21SURC/S530-A3/TR8"/>
-<part name="R5" library="Actuator Circle" deviceset="RES-0402" device="" package3d_urn="urn:adsk.eagle:package:10872901/3" value="1K"/>
+<part name="R5" library="resistor" library_urn="urn:adsk.eagle:library:348" deviceset="R-EU_" device="R0603" package3d_urn="urn:adsk.eagle:package:23555/3" value="1K"/>
 <part name="C2" library="Actuator Circle" deviceset="CAP-0603-22UF-10V-MLCC" device="" package3d_urn="urn:adsk.eagle:package:10872909/3" value="0.1uf"/>
 <part name="5V" library="Actuator Circle" deviceset="LED" device="CHIPLED_0805" package3d_urn="urn:adsk.eagle:package:15821/2" value="17-21SURC/S530-A3/TR8"/>
-<part name="R6" library="Actuator Circle" deviceset="RES-0402" device="" package3d_urn="urn:adsk.eagle:package:10872901/3" value="2k"/>
+<part name="R6" library="resistor" library_urn="urn:adsk.eagle:library:348" deviceset="R-EU_" device="R0603" package3d_urn="urn:adsk.eagle:package:23555/3" value="2k"/>
 </parts>
 <sheets>
